File: KiCad/SDBox.sch (KiCad schematic (older format))
At the start: 19 parts, among them J1 DB25_Male, J2 Micro_SD_Card_Socket, J3 Conn_01x05, U1 Rapberry_Pi_Pico_2W, U2 SN74CBT16210

Commit message: Add push button to GPIO13, remove JP1 and connect /RESET directly to RUN, change to 0603 SMD LED diodes, change resistor values on R1,R2 to 1k Ohm, move J3 to not interfere with USB-cable, bump revision to 3C
Parts:
- removed JP1: Jumper_2_Open, Connector_PinHeader_2.54mm:PinHeader_1x02_P2.54mm_Vertical, symbol Jumper:Jumper_2_Open
- added BT1: SW_Push, SDBox:Sunrom_Tactile_Switch_3x4x2mm_SMD_2-Pin, symbol Switch:SW_Push
- D1, D2: footprint LED_THT:LED_Rectangular_W5.0mm_H2.0mm -> Diode_SMD:D_0603_1608Metric_Pad1.05x0.95mm_HandSolder
- R1: value 4.7k -> 1k
- R2: value 220 -> 1k
Connections:
- net RUN is gone; now on net RESET_3V3: U1.30 (RUN)
- net GND: now also BT1.1
- net UART0_RX: now also BT1.2
Changed lines of the file:
@@
 F 0 "D1" V 8889 3033 50  0000 R CNN
 F 1 "Power LED indicator" V 8798 3033 50  0000 R CNN
-F 2 "LED_THT:LED_Rectangular_W5.0mm_H2.0mm" H 8850 3150 50  0001 C CNN
+F 2 "Diode_SMD:D_0603_1608Metric_Pad1.05x0.95mm_HandSolder" H 8850 3150 50  0001 C CNN
 F 3 "~" H 8850 3150 50  0001 C CNN
 	1    8850 3150
@@
 P 8850 2900
 F 0 "R1" H 8700 2900 50  0000 L CNN
-F 1 "4.7k" H 8900 2900 50  0000 L CNN
+F 1 "1k" H 8900 2900 50  0000 L CNN
 F 2 "Resistor_SMD:R_0805_2012Metric_Pad1.15x1.40mm_HandSolder" H 8850 2900 50  0001 C CNN
 F 3 "~" H 8850 2900 50  0001 C CNN
@@
 Text GLabel 4800 5100 0    50   Input ~ 0
 STROBE_3V3
-Text GLabel 6300 3650 1    50   Input ~ 0
+Text GLabel 5800 4300 2    50   Input ~ 0
 RESET_3V3
 Text GLabel 3750 3050 2    50   Input ~ 0
@@
 F 0 "D2" V 9100 5050 50  0000 R CNN
 F 1 "Activity LED indicator" V 9250 5150 50  0000 R CNN
-F 2 "LED_THT:LED_Rectangular_W5.0mm_H2.0mm" H 9100 4850 50  0001 C CNN
+F 2 "Diode_SMD:D_0603_1608Metric_Pad1.05x0.95mm_HandSolder" H 9100 4850 50  0001 C CNN
 F 3 "~" H 9100 4850 50  0001 C CNN
 	1    9100 4850
@@
 P 9100 4300
 F 0 "R2" H 9000 4300 50  0000 C CNN
-F 1 "220" H 9250 4300 50  0000 C CNN
+F 1 "1k" H 9250 4300 50  0000 C CNN
 F 2 "Resistor_SMD:R_0805_2012Metric_Pad1.15x1.40mm_HandSolder" H 9100 4300 50  0001 C CNN
 F 3 "~" H 9100 4300 50  0001 C CNN
@@
 Text GLabel 5800 3900 2    50   Output ~ 0
 ACT_LED
-$Comp
-L Jumper:Jumper_2_Open JP1
-U 1 1 6466A6DB
-P 6300 3850
-F 0 "JP1" V 6346 3762 50  0000 R CNN
-F 1 "Jumper_2_Open" H 6250 3700 50  0000 R CNN
-F 2 "Connector_PinHeader_2.54mm:PinHeader_1x02_P2.54mm_Vertical" H 6300 3850 50  0001 C CNN
-F 3 "~" H 6300 3850 50  0001 C CNN
-	1    6300 3850
-	0    -1   -1   0
-$EndComp
 Wire Notes Line
 	8400 3750 8400 5950
@@
 Text GLabel 4650 5850 1    50   Input ~ 0
 VCC
-Wire Wire Line
-	5800 4300 6300 4300
-Wire Wire Line
-	6300 4300 6300 4050
-Text Label 6050 4300 0    50   ~ 0
-RUN
 Text GLabel 7650 3600 1    50   Input ~ 0
 NC1
@@
 Text GLabel 3000 6200 3    50   Input ~ 0
 UART0_RX
+$Comp
+L Switch:SW_Push BT1
+U 1 1 6965AEA0
+P 7400 6100
+F 0 "BT1" H 7400 6385 50  0000 C CNN
+F 1 "SW_Push" H 7400 6294 50  0000 C CNN
+F 2 "SDBox:Sunrom_Tactile_Switch_3x4x2mm_SMD_2-Pin" H 7400 6300 50  0001 C CNN
+F 3 "~" H 7400 6300 50  0001 C CNN
+	1    7400 6100
+	1    0    0    -1
+$EndComp
+Text GLabel 7200 6100 0    50   Input ~ 0
+GND
+Text GLabel 7600 6100 2    50   Input ~ 0
+UART0_RX
 $EndSCHEMATC
